Commit message: update

File: mini_bdx/robots/bdx/robot.urdf (robot description, URDF)
Before this commit: robot onshape, 18 links, 17 joints
Links:
- removed link head_front
- added link head, mass 1e-9
- link body_module: mass 0.37223434038043856642 -> 0.37223434038043867744
- link double_u_module: mass 0.0166732881110219118 -> 0.01667328811102191527
- link double_u_module_2: mass 0.0166732881110219118 -> 0.01667328811102191527
- link head_assembly: mass 0.16975667017560497341 -> 0.16975354517560506395
- link head_link: mass 0.021984415624223832553 -> 0.021984415624223825614
- link left_hip_pitch_roll_module: mass 0.051958418033162222238 -> 0.051958418033162229177
- link leg_module: mass 0.032944425271424632173 -> 0.032944425271424639112
- link leg_module_2: mass 0.032944425271424632173 -> 0.032944425271424639112
- link leg_module_3: mass 0.032944425271424632173 -> 0.032944425271424639112
- link leg_module_4: mass 0.032944425271424632173 -> 0.032944425271424639112
- link right_hip_pitch_roll_module: mass 0.051958418033162222238 -> 0.051958418033162229177
Joints:
- removed joint head_front_frame
- added joint head_frame: type fixed, parent head_assembly, child head, origin xyz=-7.6327832942979512154e-17 8.6736173798840354721e-19 -0.0074000000000000731859 rpy=-3.141592653589793116 2.4849118514469898508e-29 -5.9944177452792396693e-27, axis 0 0 0

Commit message: update

File: mini_bdx/robots/bdx/robot.urdf (robot description, URDF)
Before this commit: robot onshape, 18 links, 17 joints
Links:
- removed link left_foot_tip
- removed link right_foot_tip
- added link left_foot, mass 1e-9
- added link right_foot, mass 1e-9
- link body_module: mass 0.37223434038043867744 -> 1.0982675034326250252; geometry collision mesh filename=package:///39281023.prt.stl; collision mesh filename=package:///bno055.stl
- link double_u_module: mass 0.01667328811102191527 -> 0.018818301231819770797
- link double_u_module_2: mass 0.01667328811102191527 -> 0.018818301231819770797
- link foot_module: mass 0.051710092735949994558 -> 0.050192424017228398636
- link foot_module_2: mass 0.051710092735949994558 -> 0.050192424017228398636
- link head_assembly: mass 0.16975354517560506395 -> 0.16981152778281508042; geometry collision mesh filename=package:///dc15_a01_horn_idle2_dummy.stl; collision mesh filename=package:///head.stl
- link head_link: mass 0.021984415624223825614 -> 0.020865926048949740013; geometry collision mesh filename=package:///axis_to_axis.stl; collision mesh filename=package:///axis_to_axis.stl
- link head_pitch_yaw: mass 0.035531283067773151985 -> 0.056026571436010752514; geometry collision mesh filename=package:///dc15_a01_case_b_dummy.stl; collision mesh filename=package:///dc15_a01_case_b_dummy.stl
- link left_hip_pitch_roll_module: mass 0.051958418033162229177 -> 0.050936078435093665173
- link leg_module: mass 0.032944425271424639112 -> 0.034530807353386039349; geometry collision mesh filename=package:///block_to_axis.stl; collision mesh filename=package:///block_to_axis.stl
- link leg_module_2: mass 0.032944425271424639112 -> 0.034530807353386039349; geometry collision mesh filename=package:///block_to_axis.stl; collision mesh filename=package:///block_to_axis.stl
- link leg_module_3: mass 0.032944425271424639112 -> 0.034530807353386039349; geometry collision mesh filename=package:///block_to_axis.stl; collision mesh filename=package:///block_to_axis.stl
- link leg_module_4: mass 0.032944425271424639112 -> 0.034530807353386039349; geometry collision mesh filename=package:///block_to_axis.stl; collision mesh filename=package:///block_to_axis.stl
- link right_hip_pitch_roll_module: mass 0.051958418033162229177 -> 0.050685765935093662904
Joints:
- removed joint head_pitch1
- removed joint head_pitch2
- removed joint left_foot_tip_frame
- removed joint right_foot_tip_frame
- added joint head_pitch: type revolute, parent head_link, child head_pitch_yaw, origin xyz=3.4694469519536141888e-18 -0.064999999999999141798 3.4694469519536141888e-18 rpy=3.1415926535897926719 -1.6569800610870191142e-15 -1.570796326794896336, axis 0 0 1, limit lower=-0.69813170079773179122 upper=0.69813170079773179122 effort=1 velocity=20
- added joint left_foot_frame: type fixed, parent foot_module_2, child left_foot, origin xyz=-0.037499999999999367173 0.0050000000000035302664 0.011500000000004340084 rpy=1.5707963267948952257 -1.1420177484200466381e-14 1.5707963267948961139, axis 0 0 0
- added joint neck_pitch: type revolute, parent body_module, child head_link, origin xyz=0.03062710048502576346 -0.018103896430577137711 0.055078922950960805538 rpy=-1.570796326794881459 -6.2505556286397272481e-14 1.0547118733946938852e-15, axis 0 0 1, limit lower=-1.3089969389957472057 upper=0.1745329251994329478 effort=1 velocity=20
- added joint right_foot_frame: type fixed, parent foot_module, child right_foot, origin xyz=-0.037499999999999200639 5.9047818717905542485e-15 0.011500000000038132497 rpy=1.5707963267948952257 -8.2376847691336273066e-15 1.57079632679489678, axis 0 0 0
- joint head_frame: origin xyz=-7.6327832942979512154e-17 8.6736173798840354721e-19 -0.0074000000000000731859 rpy=-3.141592653589793116 2.4849118514469898508e-29 -5.9944177452792396693e-27 -> xyz=-7.9797279894933126343e-17 8.6736173798840354721e-19 -0.0076000000000000789147 rpy=-3.141592653589793116 1.3183898417348306489e-16 -2.0261749666996487726e-26
- joint head_yaw: origin xyz=0.037999999999999575784 2.7755575615628913511e-17 -0.01150000000000000501 rpy=1.57079632679489678 2.7183456742966672707e-16 -1.570796326794896558 -> xyz=0.037999999999999423128 3.4694469519536141888e-17 -0.011500000000000006745 rpy=1.570796326794896558 1.5530065672147715551e-15 -1.570796326794896558
- joint left_ankle: origin xyz=-0.064999999999999738542 1.6044023748440494614e-15 8.6736173798840354721e-16 rpy=-1.1268763699943687011e-14 1.530147876329310037e-14 -3.7007434154172122983e-16 -> xyz=-0.065000000000000154876 1.6067876196235175712e-15 8.6042284408449631883e-16 rpy=-1.1368826724137153788e-14 1.6596211705633574847e-14 -2.1322488822902390562e-14
- joint left_hip_pitch: origin xyz=0.025000000000000473233 -0.0015000000000000013323 -0.0095000000000003380352 rpy=-1.5707963267948956698 7.8207331051164842944e-08 3.141592653589793116 -> xyz=0.025000000000000459355 -0.0015000000000000152101 -0.0095000000000003380352 rpy=-1.57079632679489678 7.8207331219164669488e-08 -3.141592653589793116
- joint left_hip_roll: origin xyz=0.034000000000000807354 -0.0115000000000000345 0.011500000000000017153 rpy=1.570796326794896558 -1.570796326794881681 0 -> xyz=0.034000000000001175116 -0.0115000000000000345 0.011499999999999996336 rpy=1.570796326794896558 -1.570796326794896558 0
- joint left_hip_yaw: origin xyz=0.00012710048502768600998 0.018396103569423397778 0.023078922950960308741 rpy=3.1415926535897309435 -1.5078389055347532112e-14 1.5707963267948974462 -> xyz=0.00012710048502761662104 0.018396103569423387369 0.023078922950960294863 rpy=3.1415926535897309435 -1.5078389055347532112e-14 1.5707963267948974462
- joint left_knee: origin xyz=-0.064999999999998614442 -1.7347234759768070944e-18 -9.9920072216264088638e-16 rpy=4.9960035007571566733e-16 -1.5046174721125420955e-14 -7.8207331051164856179e-08 -> xyz=-0.064999999999998281375 -6.7220534694101274908e-17 0 rpy=5.970893051203023059e-16 -1.4853578868213746426e-14 -7.8207310266750229308e-08
- joint right_ankle: origin xyz=-0.065000000000002153278 -8.8752789839663392968e-16 1.8041124150158793782e-16 rpy=-1.0269562977782461341e-14 1.7185939463948808782e-15 1.0613769886213497671e-13 -> xyz=-0.065000000000002028377 -8.9902044142498027668e-16 1.249000902703301108e-16 rpy=-1.0269562977784517112e-14 1.8977874827185263815e-15 1.0627453601663781033e-13
- joint right_hip_pitch: origin xyz=0.025000000000000216493 -0.024499999999999855227 -0.013499999999999812497 rpy=1.570796326794896558 2.7235158572835087452e-16 -3.141592653589793116 -> xyz=0.025000000000000216493 -0.024499999999999855227 -0.013499999999999812497 rpy=1.5707963267948970021 -8.3130108030798317137e-14 -3.1415926535897913396
- joint right_hip_roll: origin xyz=-0.033999999999999877542 0.011500000000001705039 0.011500000000000806452 rpy=-1.570796326794896336 -1.5707963267948286123 0 -> xyz=-0.033999999999999905298 0.011499999999999989397 0.011499999999999895722 rpy=-1.5707963267948961139 -1.570796326794896336 0
- joint right_hip_yaw: origin xyz=0.00012710048502772764334 -0.031603896430576608467 0.023078922950959552401 rpy=3.1415926535897304994 -1.5078389055347532112e-14 1.5707963267948974462 -> xyz=0.00012710048502765998913 -0.031603896430576622345 0.023078922950959545463 rpy=3.1415926535897304994 -1.5078389055347532112e-14 1.5707963267948974462
- joint right_knee: origin xyz=-0.065000000000000626721 -2.0578157233774874157e-16 2.498001805406602216e-16 rpy=-8.5052035001972290279e-16 1.421728862755529065e-14 -1.0522870376072329388e-13 -> xyz=-0.065000000000000640599 -1.9689111452336760522e-16 -5.5511151231257827021e-17 rpy=1.1589216316011910219e-16 -2.0968964649445356432e-15 -1.2051470932306016186e-13
- joint trunk_frame: origin xyz=-0.014872899514971796298 -0.0066038964305765012613 0.015078922950959212229 rpy=1.5111348801390842167e-14 -6.2433989600656073464e-14 9.1593399531630240418e-16 -> xyz=0.03252710048502828466 -0.0066038964305764136578 0.012578922950962063629 rpy=1.5074919608395890887e-14 -6.236720274683202662e-14 9.4368957093184533185e-16

Commit message: update

File: mini_bdx/robots/bdx/robot.urdf (robot description, URDF)
Before this commit: robot onshape, 18 links, 17 joints
Links:
- link body_module: mass 1.0982675034326250252 -> 0.49727524155661395611; geometry collision mesh filename=package:///39281023.prt.stl; collision mesh filename=package:///bno055.stl
- link foot_module: mass 0.050192424017228398636 -> 0.028234070013912714731
- link foot_module_2: mass 0.050192424017228398636 -> 0.028234070013912714731
- link head_assembly: mass 0.16981152778281508042 -> 0.089584351569467951526
- link head_link: mass 0.020865926048949740013 -> 0.020865926048949729604
- link head_pitch_yaw: mass 0.056026571436010752514 -> 0.055748483731440375
Joints:
- joint head_pitch: origin xyz=3.4694469519536141888e-18 -0.064999999999999141798 3.4694469519536141888e-18 rpy=3.1415926535897926719 -1.6569800610870191142e-15 -1.570796326794896336 -> xyz=3.4694469519536141888e-18 -0.064999999999999114042 3.4694469519536141888e-18 rpy=3.1415926535897926719 -1.6569800610870191142e-15 -1.570796326794896336
- joint left_ankle: origin xyz=-0.065000000000000154876 1.6067876196235175712e-15 8.6042284408449631883e-16 rpy=-1.1368826724137153788e-14 1.6596211705633574847e-14 -2.1322488822902390562e-14 -> xyz=-0.065000000000000140998 1.6111244283134595889e-15 8.7430063189231077558e-16 rpy=-1.1368826724137153788e-14 1.6596211705633574847e-14 -2.1322488822902390562e-14
- joint left_foot_frame: origin xyz=-0.037499999999999367173 0.0050000000000035302664 0.011500000000004340084 rpy=1.5707963267948952257 -1.1420177484200466381e-14 1.5707963267948961139 -> xyz=-0.037499999999999339417 0.0050000000000035302664 0.011500000000004333145 rpy=1.5707963267948952257 -1.1420177484200466381e-14 1.5707963267948961139
- joint left_hip_pitch: origin xyz=0.025000000000000459355 -0.0015000000000000152101 -0.0095000000000003380352 rpy=-1.57079632679489678 7.8207331219164669488e-08 -3.141592653589793116 -> xyz=0.025000000000000459355 -0.0015000000000000013323 -0.0095000000000003380352 rpy=-1.57079632679489678 7.8207331219164669488e-08 -3.141592653589793116
- joint left_hip_roll: limit lower=-1.570796326794896558 upper=0.34906585039886589561 effort=1 velocity=20 -> lower=-1.570796326794896558 upper=0.43633231299858238339 effort=1 velocity=20; origin xyz=0.034000000000001175116 -0.0115000000000000345 0.011499999999999996336 rpy=1.570796326794896558 -1.570796326794896558 0 -> xyz=0.034000000000001168177 -0.0115000000000000345 0.011499999999999996336 rpy=1.570796326794896558 -1.570796326794896558 0
- joint left_hip_yaw: origin xyz=0.00012710048502761662104 0.018396103569423387369 0.023078922950960294863 rpy=3.1415926535897309435 -1.5078389055347532112e-14 1.5707963267948974462 -> xyz=0.00012710048502760968214 0.018396103569423397778 0.023078922950960291394 rpy=3.1415926535897309435 -1.5078389055347532112e-14 1.5707963267948974462
- joint left_knee: origin xyz=-0.064999999999998281375 -6.7220534694101274908e-17 0 rpy=5.970893051203023059e-16 -1.4853578868213746426e-14 -7.8207310266750229308e-08 -> xyz=-0.064999999999998281375 -5.8763757748714340323e-17 0 rpy=5.970893051203023059e-16 -1.4853578868213746426e-14 -7.8207310266750229308e-08
- joint neck_pitch: origin xyz=0.03062710048502576346 -0.018103896430577137711 0.055078922950960805538 rpy=-1.570796326794881459 -6.2505556286397272481e-14 1.0547118733946938852e-15 -> xyz=0.030627100485025756521 -0.018103896430577130772 0.055078922950960805538 rpy=-1.570796326794881459 -6.2505556286397272481e-14 1.0547118733946938852e-15
- joint right_ankle: origin xyz=-0.065000000000002028377 -8.9902044142498027668e-16 1.249000902703301108e-16 rpy=-1.0269562977784517112e-14 1.8977874827185263815e-15 1.0627453601663781033e-13 -> xyz=-0.0650000000000020145 -9.0595933532888750506e-16 1.3877787807814456755e-16 rpy=-1.0269562978010203906e-14 7.7715611723723191114e-16 2.0455945828244817402e-14
- joint right_foot_frame: origin xyz=-0.037499999999999200639 5.9047818717905542485e-15 0.011500000000038132497 rpy=1.5707963267948952257 -8.2376847691336273066e-15 1.57079632679489678 -> xyz=-0.037499999999998978595 -3.5605199344423965613e-16 0.011499999999999552247 rpy=1.5707963267948954478 -9.9920072216264293742e-15 1.57079632679489678
- joint right_hip_pitch: origin xyz=0.025000000000000216493 -0.024499999999999855227 -0.013499999999999812497 rpy=1.5707963267948970021 -8.3130108030798317137e-14 -3.1415926535897913396 -> xyz=0.025000000000000646705 -0.024500000000000743405 -0.013499999999999783007 rpy=1.5707963267948972241 -9.4876329561990965088e-14 -3.141592653589793116
- joint right_hip_roll: limit lower=-1.570796326794896558 upper=0.34906585039886589561 effort=1 velocity=20 -> lower=-1.570796326794896558 upper=0.43633231299858238339 effort=1 velocity=20; origin xyz=-0.033999999999999905298 0.011499999999999989397 0.011499999999999895722 rpy=-1.5707963267948961139 -1.570796326794896336 0 -> xyz=-0.033999999999999905298 0.011499999999999989397 0.011499999999999895722 rpy=-1.5707963267948958919 -1.570796326794896336 0
- joint right_hip_yaw: origin xyz=0.00012710048502765998913 -0.031603896430576622345 0.023078922950959545463 rpy=3.1415926535897304994 -1.5078389055347532112e-14 1.5707963267948974462 -> xyz=0.00012710048502765305023 -0.031603896430576608467 0.023078922950959548932 rpy=3.1415926535897304994 -1.5078389055347532112e-14 1.5707963267948974462
- joint right_knee: origin xyz=-0.065000000000000640599 -1.9689111452336760522e-16 -5.5511151231257827021e-17 rpy=1.1589216316011910219e-16 -2.0968964649445356432e-15 -1.2051470932306016186e-13 -> xyz=-0.065000000000000890399 -1.8409752888803865289e-16 2.3592239273284576484e-16 rpy=1.1102230529243367767e-16 2.2204460492507932999e-16 -1.1500818382616808057e-13
- joint trunk_frame: origin xyz=0.03252710048502828466 -0.0066038964305764136578 0.012578922950962063629 rpy=1.5074919608395890887e-14 -6.236720274683202662e-14 9.4368957093184533185e-16 -> xyz=0.032527100485028291599 -0.0066038964305764145252 0.012578922950962011587 rpy=1.5111348801390835856e-14 -6.2433989600656048221e-14 9.1593399531630240418e-16

Commit message: update

File: mini_bdx/robots/bdx/robot.urdf (robot description, URDF)
Before this commit: robot onshape, 18 links, 17 joints
Links:
- added link left_antenna_assembly, mass 0.0021739976315290265516; collision mesh filename=package:///antenna.stl; collision mesh filename=package:///antenna_holder_left.stl
- added link right_antenna_assembly, mass 0.0021739987496008352993; collision mesh filename=package:///antenna.stl; collision mesh filename=package:///antenna_holder_right.stl
- link body_module: mass 0.49727524155661395611 -> 0.50186117579999178773; geometry collision mesh filename=package:///39281023.prt.stl; collision mesh filename=package:///bms.stl
- link foot_module: mass 0.028234070013912714731 -> 0.028234070013912770242
- link foot_module_2: mass 0.028234070013912714731 -> 0.028234070013912770242
- link head_assembly: mass 0.089584351569467951526 -> 0.11182196316230802458; geometry collision mesh filename=package:///antenna_motor_holder.stl; collision mesh filename=package:///antenna_motor_holder.stl
- link head_link: mass 0.020865926048949729604 -> 0.020865926048949740013
Joints:
- added joint left_antenna: type revolute, parent head_assembly, child left_antenna_assembly, origin xyz=-0.052000000000000864975 -0.03151836494610388284 0.0098000000000001419309 rpy=-1.57079632679489678 1.1974744221533701829e-16 1.1102230247078030323e-16, axis 0 0 1, limit lower=-1.1344640137963142301 upper=2.0943951023931952626 effort=1 velocity=20
- added joint right_antenna: type revolute, parent head_assembly, child right_antenna_assembly, origin xyz=-0.052000000000000719258 0.031518364946103966107 0.0098000000000001141753 rpy=1.570796326794896558 1.1974744221538782586e-16 5.5511151224369080677e-17, axis 0 0 1, limit lower=-2.0943951023931952626 upper=1.1344640137963142301 effort=1 velocity=20

Commit message: update

File: mini_bdx/robots/bdx/robot.urdf (robot description, URDF)
Before this commit: robot BDX, 20 links, 19 joints
Links:
- link head_assembly: mass 0.11182196316230802458 -> 0.11182196316230799682
- link head_link: mass 0.020865926048949740013 -> 0.020865926048949733074
- link left_antenna_assembly: mass 0.0021739976315290265516 -> 0.0021739976315290274189
- link right_antenna_assembly: mass 0.0021739987496008352993 -> 0.0021739987496008348657
Joints:
- joint head_frame: origin xyz=-7.9797279894933126343e-17 8.6736173798840354721e-19 -0.0076000000000000789147 rpy=-3.141592653589793116 1.3183898417348306489e-16 -2.0261749666996487726e-26 -> xyz=-5.898059818321144121e-17 -1.7347234759768070944e-18 -0.0076000000000001344258 rpy=3.141592653589793116 1.1974744221542317669e-16 1.1102230247078422288e-16
- joint head_yaw: origin xyz=0.037999999999999423128 3.4694469519536141888e-17 -0.011500000000000006745 rpy=1.570796326794896558 1.5530065672147715551e-15 -1.570796326794896558 -> xyz=0.037999999999999423128 3.4694469519536141888e-17 -0.011500000000000006745 rpy=1.570796326794896558 1.6085177185030839443e-15 -1.570796326794896558
- joint left_antenna: origin xyz=-0.052000000000000864975 -0.03151836494610388284 0.0098000000000001419309 rpy=-1.57079632679489678 1.1974744221533701829e-16 1.1102230247078030323e-16 -> xyz=-0.052000000000000962119 -0.031518364946103889779 0.0098000000000001419309 rpy=-1.57079632679489678 1.1974744221543518216e-16 1.6653345375909212544e-16
- joint left_foot_frame: origin xyz=-0.037499999999999339417 0.0050000000000035302664 0.011500000000004333145 rpy=1.5707963267948952257 -1.1420177484200466381e-14 1.5707963267948961139 -> xyz=-0.037499999999999256151 -5.2475385148298414606e-17 0.011499999999999850619 rpy=1.5707963267948954478 -9.9737163921664587049e-15 1.570796326794896558
- joint right_ankle: origin xyz=-0.0650000000000020145 -9.0595933532888750506e-16 1.3877787807814456755e-16 rpy=-1.0269562978010203906e-14 7.7715611723723191114e-16 2.0455945828244817402e-14 -> xyz=-0.065000000000002070011 -9.0726037793587011038e-16 1.249000902703301108e-16 rpy=-1.028864493624538396e-14 7.7715611723731079723e-16 2.0438598593485175549e-14
- joint right_antenna: origin xyz=-0.052000000000000719258 0.031518364946103966107 0.0098000000000001141753 rpy=1.570796326794896558 1.1974744221538782586e-16 5.5511151224369080677e-17 -> xyz=-0.052000000000000809464 0.031518364946103966107 0.0098000000000001419309 rpy=1.570796326794896558 1.1974744221548598974e-16 1.1102230251268074882e-16
- joint right_foot_frame: origin xyz=-0.037499999999998978595 -3.5605199344423965613e-16 0.011499999999999552247 rpy=1.5707963267948954478 -9.9920072216264293742e-15 1.57079632679489678 -> xyz=-0.037499999999999034106 -6.6570013390609972248e-17 0.011499999999999982458 rpy=1.5707963267948954478 -9.9920072216265019494e-15 1.570796326794896558
- joint trunk_frame: origin xyz=0.032527100485028291599 -0.0066038964305764145252 0.012578922950962011587 rpy=1.5111348801390835856e-14 -6.2433989600656048221e-14 9.1593399531630240418e-16 -> xyz=0.032527100485028298538 -0.0066038964305764145252 0.012578922950962011587 rpy=1.5111348801390835856e-14 -6.2433989600656048221e-14 9.1593399531630240418e-16
