Commit message: placo walk open loop

File: mini_bdx/robots/open_duck_mini_v2/robot.urdf (robot description, URDF)
Before this commit: robot onshape, 14 links, 13 joints
Links:
- removed link left_ankle_pitch_assembly
- removed link left_foot_assembly
- removed link left_hip_pitch_assembly
- removed link left_hip_roll_assembly
- removed link left_knee_pitch_assembly
- removed link right_ankle_pitch_assembly
- removed link right_foot_assembly
- removed link right_hip_pitch_assembly
- removed link right_hip_roll_assembly
- removed link right_knee_pitch_assembly
- added link foot_assembly, mass 0.056240000000000012204; collision mesh filename=package:///foot_bottom.stl; collision mesh filename=package:///foot_side.stl
- added link foot_assembly_2, mass 0.056240000000000012204; collision mesh filename=package:///foot_bottom.stl; collision mesh filename=package:///foot_side.stl
- added link head, mass 1e-9
- added link head_assembly, mass 0.22929000000000004933; collision mesh filename=package:///head.stl; collision mesh filename=package:///head_bot_sheet.stl
- added link head_pitch_assembly, mass 0.071850000000000024958; collision mesh filename=package:///drive_palonier.stl; collision mesh filename=package:///head_pitch_to_yaw.stl
- added link hip_roll_assembly, mass 0.066480000000000011307; collision mesh filename=package:///drive_palonier.stl; collision mesh filename=package:///passive_palonier.stl
- added link hip_roll_assembly_2, mass 0.066480000000000011307; collision mesh filename=package:///drive_palonier.stl; collision mesh filename=package:///passive_palonier.stl
- added link knee_and_ankle_assembly, mass 0.12406999999999994422; collision mesh filename=package:///drive_palonier.stl; collision mesh filename=package:///left_cache.stl
- added link knee_and_ankle_assembly_2, mass 0.072590000000000015623; collision mesh filename=package:///drive_palonier.stl; collision mesh filename=package:///left_knee_to_ankle_left_sheet.stl
- added link knee_and_ankle_assembly_3, mass 0.12407000000000002748; collision mesh filename=package:///drive_palonier.stl; collision mesh filename=package:///left_knee_to_ankle_left_sheet.stl
- added link knee_and_ankle_assembly_4, mass 0.072590000000000015623; collision mesh filename=package:///drive_palonier.stl; collision mesh filename=package:///left_knee_to_ankle_left_sheet.stl
- added link left_roll_to_pitch_assembly, mass 0.075160000000000018461; collision mesh filename=package:///drive_palonier.stl; collision mesh filename=package:///left_roll_to_pitch.stl
- added link neck_assembly, mass 0.066180000000000016591; collision mesh filename=package:///drive_palonier.stl; collision mesh filename=package:///neck_left_sheet.stl
- added link right_roll_to_pitch_assembly, mass 0.075160000000000018461; collision mesh filename=package:///drive_palonier.stl; collision mesh filename=package:///passive_palonier.stl
- link trunk_assembly: mass 0.22534624917253631704 -> 0.55922072109020470876; geometry collision mesh filename=package:///body_back.stl; collision mesh filename=package:///body_front.stl
Joints:
- added joint head_frame: type fixed, parent head_assembly, child head, origin xyz=4.1633363423443370266e-17 0 -0.01249999999999990008 rpy=-3.1415926535897797933 4.3716373664754018489e-18 7.4988647406086779923e-30, axis 0 0 0
- added joint head_pitch: type revolute, parent neck_assembly, child head_pitch_assembly, origin xyz=1.0408340855860842566e-16 0.066000000000000391687 -3.4694469519536141888e-18 rpy=-1.0915849447069766081e-16 -7.3845547632106068786e-17 -1.0417200973690603325e-16, axis 0 0 1, limit lower=-1.570796326794896558 upper=1.570796326794896558 effort=1 velocity=20
- added joint head_yaw: type revolute, parent head_pitch_assembly, child head_assembly, origin xyz=-2.0816681711721685133e-17 0.056900000000000033884 0.019049999999999952388 rpy=1.5707963267948958919 -2.9140480977164958126e-15 -8.9523033089878119206e-15, axis 0 0 1, limit lower=-2.9670597283903603625 upper=2.9670597283903603625 effort=1 velocity=20
- added joint neck_pitch: type revolute, parent trunk_assembly, child neck_assembly, origin xyz=-0.035437537550831413324 0.012752766445331959258 0.068008119366846808695 rpy=1.5707963267948341635 0.021825623709755184038 1.3218913913091132832e-13, axis 0 0 1, limit lower=-0.34906585039886589561 upper=1.1344640137963142301 effort=1 velocity=20
- joint left_ankle: child left_foot_assembly -> foot_assembly; origin xyz=-4.1633363423443370266e-17 -0.1121850000000000902 -5.5511151231257827021e-17 rpy=-8.5765521874236585977e-33 1.2325951644078325881e-32 1.0571416753509825153e-64 -> xyz=0 -0.07865000000000006708 9.9999999999988986588e-05 rpy=-5.5077724532749743024e-16 9.2653469445928301633e-16 3.2402024558001311503e-14; parent left_ankle_pitch_assembly -> knee_and_ankle_assembly_2
- joint left_foot_frame: origin xyz=-2.724806148598352129e-05 -0.053059999999999940545 0.019049999999999955858 rpy=-1.570796326794896558 2.9705808733109505824e-68 -1.9698832702909219349e-42 -> xyz=0 -0.036724999999999979883 0.019049999999999983613 rpy=-1.570796326794896558 -3.4146152368508307717e-19 -1.8519077370852487142e-17; parent left_foot_assembly -> foot_assembly
- joint left_hip_pitch: child left_knee_pitch_assembly -> knee_and_ankle_assembly; origin xyz=0.079149999999999831601 9.9999999997255062389e-06 0.039456000000000025774 rpy=-3.1415926535897913396 1.5707963267948958919 0 -> xyz=0.074149999999998272848 1.249000902703301108e-15 0.035109999999998510456 rpy=3.1415926535897926719 1.5707963267948574781 0; parent left_hip_pitch_assembly -> left_roll_to_pitch_assembly
- joint left_hip_roll: child left_hip_pitch_assembly -> left_roll_to_pitch_assembly; origin xyz=0.019149999999999948314 6.0999999999970799802e-05 -0.016950000000000201017 rpy=-1.5707963267948958919 -6.9295263485299483695e-30 1.570796326794896336 -> xyz=0.019050000000002648148 1.9602375278537920167e-15 -0.046015000000004538383 rpy=-1.5707963267950215691 1.6937530152664249305e-13 1.5707963267952902431; parent left_hip_roll_assembly -> hip_roll_assembly
- joint left_hip_yaw: child left_hip_roll_assembly -> hip_roll_assembly; limit lower=-0.785398163397448279 upper=0.785398163397448279 effort=1 velocity=20 -> lower=-0.52359877559829881566 upper=0.52359877559829881566 effort=1 velocity=20; origin xyz=1.3739009929736358287e-17 0.054995999999999753416 -0.019049999999999990552 rpy=3.5632986684149037817e-32 7.8886090522100865249e-31 -7.3955709864469561171e-32 -> xyz=-0.056394334796673495358 0.028602766445326346934 0.024395090932709764808 rpy=-6.2403804745132919901e-14 0.021825623709755430368 1.3218914061185209833e-13
- joint left_knee: child left_ankle_pitch_assembly -> knee_and_ankle_assembly_2; limit lower=-0.52359877559829881566 upper=2.1816615649929120835 effort=1 velocity=20 -> lower=-1.570796326794896558 upper=1.570796326794896558 effort=1 velocity=20; origin xyz=2.4286128663675299322e-17 -0.1123160000000001657 -9.9999999999794697558e-05 rpy=-1.7763568394002528313e-15 -0 2.1895288505075266733e-47 -> xyz=-9.7144514654701197287e-17 -0.078649999999999734013 9.9999999999961231012e-05 rpy=7.358361518165846965e-16 5.0845139115396107043e-16 -7.1846367703695162136e-14; parent left_knee_pitch_assembly -> knee_and_ankle_assembly
- joint right_ankle: child right_foot_assembly -> foot_assembly_2; origin xyz=1.3183898417423733918e-16 0.11218500000000031225 8.3266726846886740532e-17 rpy=1.4643357955393777909e-16 -1.4438978053469552301e-16 3.3321594868555283369e-16 -> xyz=-2.7755575615628913511e-17 -0.078650000000000080957 9.9999999999961231012e-05 rpy=-2.6194324489465746712e-16 2.8316471284964215798e-29 9.5878895885319479181e-14; parent right_ankle_pitch_assembly -> knee_and_ankle_assembly_4
- joint right_foot_frame: origin xyz=0.00050000000000001779132 0.053059999999999940545 0.01954999999999990079 rpy=1.570796326794896558 -4.4483193573663491162e-23 4.9409130870146903851e-32 -> xyz=-1.3877787807814456755e-17 -0.036724999999999979883 0.019049999999999969735 rpy=-1.570796326794896558 -4.7247190275601867229e-17 6.0085748048618062173e-16; parent right_foot_assembly -> foot_assembly_2
- joint right_hip_pitch: child right_knee_pitch_assembly -> knee_and_ankle_assembly_3; origin xyz=-0.079149999999999859357 9.9999999996144839365e-06 0.039455999999999782912 rpy=-1.7282771299945109835e-15 1.5707963267948958919 0 -> xyz=-0.074149999999999993694 -2.0816681711721685133e-17 0.035110000000000009257 rpy=-2.1823850769468260177e-17 1.5707963267948927832 0; parent right_hip_pitch_assembly -> right_roll_to_pitch_assembly
- joint right_hip_roll: child right_hip_pitch_assembly -> right_roll_to_pitch_assembly; origin xyz=0.019150000000000055866 -6.099999999998467759e-05 -0.016950000000000447348 rpy=-1.5707963267948943376 -2.4982621091609909182e-15 1.5707963267948898967 -> xyz=0.019050000000005999634 2.9060087669563472446e-14 -0.046014999999998154601 rpy=-1.570796326794797082 -7.3141829490872532251e-14 1.5707963267946682961; parent right_hip_roll_assembly -> hip_roll_assembly_2
- joint right_hip_yaw: child right_hip_roll_assembly -> hip_roll_assembly_2; limit lower=-0.785398163397448279 upper=0.785398163397448279 effort=1 velocity=20 -> lower=-0.52359877559829881566 upper=0.52359877559829881566 effort=1 velocity=20; origin xyz=1.6736441286736465097e-17 -0.05499600000000029465 -0.019049999999999987083 rpy=-2.4960052079258594172e-31 3.3280069439011422404e-31 -3.4615137454088894957e-07 -> xyz=-0.056394334796664107035 -0.041397233554676490797 0.024395090932713945492 rpy=-5.7479562369434986172e-14 0.021825623709755558738 3.5607454337323585543e-13
- joint right_knee: child right_ankle_pitch_assembly -> knee_and_ankle_assembly_4; limit lower=-2.1816615649929120835 upper=0.52359877559829881566 effort=1 velocity=20 -> lower=-1.570796326794896558 upper=1.570796326794896558 effort=1 velocity=20; origin xyz=4.5102810375396984455e-17 0.11231600000000015183 -9.9999999999933475436e-05 rpy=8.6413837281558197907e-18 3.2674690263357178969e-17 9.42818147085318761e-15 -> xyz=-1.360023205165816762e-15 0.07864999999999899849 0.036999999999998534062 rpy=3.141592653589793116 -5.3042305426499207572e-15 1.0017539295583627067e-13; parent right_knee_pitch_assembly -> knee_and_ankle_assembly_3
- joint trunk_frame: origin xyz=0 -2.7235158572835871382e-16 0.022500000000000019984 rpy=0 -0 0 -> xyz=-0.060471084556686989508 -0.0063972335546741820184 0.066744147727335195741 rpy=-6.3086333636868837384e-14 0.021825623709755163221 1.3209498708375492755e-13

Commit message: updated urdf and mjcf

File: mini_bdx/robots/open_duck_mini_v2/robot.urdf (robot description, URDF)
Before this commit: robot onshape, 18 links, 17 joints
Links:
- removed link head_pitch_assembly
- removed link neck_assembly
- added link head_pitch_to_yaw, mass 0.015591038955987642986; collision mesh filename=package:///head_pitch_to_yaw.stl; visual mesh filename=package:///head_pitch_to_yaw.stl
- added link left_antenna_holder, mass 0.00421628909577088061; collision mesh filename=package:///antenna.stl; collision mesh filename=package:///left_antenna_holder.stl
- added link neck_pitch_assembly, mass 0.066180000000000030469; collision mesh filename=package:///drive_palonier.stl; collision mesh filename=package:///neck_left_sheet.stl
- added link neck_yaw_assembly, mass 0.090572249204174976045; collision mesh filename=package:///drive_palonier.stl; collision mesh filename=package:///head_yaw_to_roll.stl
- added link right_antenna_holder, mass 0.004216286984950681424; collision mesh filename=package:///antenna.stl; collision mesh filename=package:///right_antenna_holder.stl
- link foot_assembly: mass 0.056240000000000012204 -> 0.075240000000000001323; geometry collision mesh filename=package:///foot_bottom_pla.stl; collision mesh filename=package:///foot_bottom_tpu.stl
- link foot_assembly_2: mass 0.056240000000000012204 -> 0.075240000000000001323; geometry collision mesh filename=package:///foot_bottom_pla.stl; collision mesh filename=package:///foot_bottom_tpu.stl
- link head_assembly: mass 0.22929000000000004933 -> 0.33587292587593409188; geometry collision mesh filename=package:///board.stl; collision mesh filename=package:///drive_palonier.stl
- link hip_roll_assembly: mass 0.066480000000000011307 -> 0.066480000000000025184
- link hip_roll_assembly_2: mass 0.066480000000000011307 -> 0.066480000000000025184
- link knee_and_ankle_assembly: mass 0.12406999999999994422 -> 0.12407000000000002748
- link knee_and_ankle_assembly_2: mass 0.072590000000000015623 -> 0.072590000000000029501
- link knee_and_ankle_assembly_4: mass 0.072590000000000015623 -> 0.072590000000000029501
- link right_roll_to_pitch_assembly: mass 0.075160000000000018461 -> 0.075160000000000032339
- link trunk_assembly: mass 0.55922072109020470876 -> 0.69443340465392744409; geometry collision mesh filename=package:///battery_pack_lid.stl; collision mesh filename=package:///bno055.stl
Joints:
- added joint head_roll: type revolute, parent neck_yaw_assembly, child head_assembly, origin xyz=0.040950000000000402745 1.1462727468602995629e-16 -0.019150000000000444444 rpy=-2.4980018054066286428e-15 -1.5707963267948730213 0, axis 0 0 1, limit lower=-0.52359877559829881566 upper=0.52359877559829881566 effort=1 velocity=20
- added joint left_antenna: type revolute, parent head_assembly, child left_antenna_holder, origin xyz=0.00070406945503787010665 0.060662837687360374184 0.11643485329544565887 rpy=3.1415926535897309435 1.3045791727887228184 1.3234423712230789505, axis 0 0 1, limit lower=-1.570796326794896558 upper=1.570796326794896558 effort=1 velocity=20
- added joint right_antenna: type revolute, parent head_assembly, child right_antenna_holder, origin xyz=0.00070406945503653783902 -0.060662837687360852967 0.11643485329544586704 rpy=-3.1415926535897518157 1.3045791727887290357 -1.3234423712230898307, axis 0 0 1, limit lower=-1.570796326794896558 upper=1.570796326794896558 effort=1 velocity=20
- joint head_frame: origin xyz=4.1633363423443370266e-17 0 -0.01249999999999990008 rpy=-3.1415926535897797933 4.3716373664754018489e-18 7.4988647406086779923e-30 -> xyz=0.042450000000000626121 -2.563053935755732482e-16 0.03595000000000117546 rpy=-1.2621774483535835759e-29 1.5707963267948756858 0
- joint head_pitch: child head_pitch_assembly -> head_pitch_to_yaw; limit lower=-1.570796326794896558 upper=1.570796326794896558 effort=1 velocity=20 -> lower=-0.785398163397448279 upper=0.785398163397448279 effort=1 velocity=20; origin xyz=1.0408340855860842566e-16 0.066000000000000391687 -3.4694469519536141888e-18 rpy=-1.0915849447069766081e-16 -7.3845547632106068786e-17 -1.0417200973690603325e-16 -> xyz=-5.6378512969246230568e-18 0.066000000000000003109 -6.9388939039072283776e-18 rpy=5.9571514509304171254e-17 -7.163548953726033378e-17 1.6653345369378257762e-16; parent neck_assembly -> neck_pitch_assembly
- joint head_yaw: child head_assembly -> neck_yaw_assembly; limit lower=-2.9670597283903603625 upper=2.9670597283903603625 effort=1 velocity=20 -> lower=-2.7925268031909271649 upper=2.7925268031909271649 effort=1 velocity=20; origin xyz=-2.0816681711721685133e-17 0.056900000000000033884 0.019049999999999952388 rpy=1.5707963267948958919 -2.9140480977164958126e-15 -8.9523033089878119206e-15 -> xyz=-1.5178830414797062076e-17 0.056999999999999939604 0.019049999999999959327 rpy=-1.570796326794896558 -7.286368982477690022e-17 -5.2678381782433861865e-15; parent head_pitch_assembly -> head_pitch_to_yaw
- joint left_ankle: origin xyz=0 -0.07865000000000006708 9.9999999999988986588e-05 rpy=-5.5077724532749743024e-16 9.2653469445928301633e-16 3.2402024558001311503e-14 -> xyz=3.8857805861880478915e-16 -0.078649999999999067879 9.9999999999947353224e-05 rpy=-3.0577093135086125731e-16 -2.1510571099027823781e-16 -1.1379786005983670304e-15
- joint left_foot_frame: origin xyz=0 -0.036724999999999979883 0.019049999999999983613 rpy=-1.570796326794896558 -3.4146152368508307717e-19 -1.8519077370852487142e-17 -> xyz=0.00049999999999996574962 -0.036224999999999646372 0.019550000000000317124 rpy=-1.570796326794896558 4.8789097759078905605e-18 3.7865323450608544239e-29
- joint left_hip_pitch: limit lower=-1.570796326794896558 upper=0.52359877559829881566 effort=1 velocity=20 -> lower=-1.2217304763960306069 upper=0.52359877559829881566 effort=1 velocity=20; origin xyz=0.074149999999998272848 1.249000902703301108e-15 0.035109999999998510456 rpy=3.1415926535897926719 1.5707963267948574781 0 -> xyz=0.074149999999998994493 5.7702594872394152858e-16 0.035109999999999731701 rpy=-3.141592653589793116 1.5707963267948958919 0
- joint left_hip_roll: origin xyz=0.019050000000002648148 1.9602375278537920167e-15 -0.046015000000004538383 rpy=-1.5707963267950215691 1.6937530152664249305e-13 1.5707963267952902431 -> xyz=0.019050000000002908357 -1.2559397966072083364e-15 -0.046015000000000465252 rpy=-1.57079632679495651 1.0208316397064496209e-13 1.5707963267945266317
- joint left_hip_yaw: origin xyz=-0.056394334796673495358 0.028602766445326346934 0.024395090932709764808 rpy=-6.2403804745132919901e-14 0.021825623709755430368 1.3218914061185209833e-13 -> xyz=-0.018999999999999715034 0.035000000000001356415 0.045940938812377457579 rpy=-5.4063708435955792693e-16 -2.1649348979904514729e-14 -1.6653345373435771223e-16
- joint left_knee: origin xyz=-9.7144514654701197287e-17 -0.078649999999999734013 9.9999999999961231012e-05 rpy=7.358361518165846965e-16 5.0845139115396107043e-16 -7.1846367703695162136e-14 -> xyz=6.2450045135165055399e-17 -0.078649999999999636868 9.9999999999988986588e-05 rpy=-1.433738720798104591e-17 9.7838404045009444717e-16 4.9960036108120734026e-16
- joint neck_pitch: child neck_assembly -> neck_pitch_assembly; origin xyz=-0.035437537550831413324 0.012752766445331959258 0.068008119366846808695 rpy=1.5707963267948341635 0.021825623709755184038 1.3218913913091132832e-13 -> xyz=0.00099999999999897046243 0.019150000000000326483 0.090000938812376238274 rpy=1.57079632679489678 -2.2148949341271863515e-14 2.5552148182455563673e-16
- joint right_ankle: origin xyz=-2.7755575615628913511e-17 -0.078650000000000080957 9.9999999999961231012e-05 rpy=-2.6194324489465746712e-16 2.8316471284964215798e-29 9.5878895885319479181e-14 -> xyz=-2.5673907444456744997e-16 -0.078649999999999331557 9.9999999999947353224e-05 rpy=3.1786111035240684541e-16 -6.6613381497353178635e-16 1.026830726893522614e-13
- joint right_foot_frame: origin xyz=-1.3877787807814456755e-17 -0.036724999999999979883 0.019049999999999969735 rpy=-1.570796326794896558 -4.7247190275601867229e-17 6.0085748048618062173e-16 -> xyz=0.00050000000000024330538 -0.036224999999999923928 0.019550000000000650191 rpy=-1.570796326794896558 -3.0222156344620005664e-28 -2.5243548967072377773e-28
- joint right_hip_pitch: limit lower=-0.52359877559829881566 upper=1.570796326794896558 effort=1 velocity=20 -> lower=-0.52359877559829881566 upper=1.2217304763960306069 effort=1 velocity=20; origin xyz=-0.074149999999999993694 -2.0816681711721685133e-17 0.035110000000000009257 rpy=-2.1823850769468260177e-17 1.5707963267948927832 0 -> xyz=-0.074149999999999938183 1.3700249702069955404e-16 0.035109999999999981501 rpy=-5.8199867801976243694e-16 1.5707963267947913089 0
- joint right_hip_roll: origin xyz=0.019050000000005999634 2.9060087669563472446e-14 -0.046014999999998154601 rpy=-1.570796326794797082 -7.3141829490872532251e-14 1.5707963267946682961 -> xyz=0.019050000000007772522 3.498590306350024548e-14 -0.046015000000001887726 rpy=-1.5707963267947930852 -7.5380278374294396407e-14 1.5707963267945495023
- joint right_hip_yaw: origin xyz=-0.056394334796664107035 -0.041397233554676490797 0.024395090932713945492 rpy=-5.7479562369434986172e-14 0.021825623709755558738 3.5607454337323585543e-13 -> xyz=-0.018999999999999697686 -0.035000000000001127431 0.045940938812377443701 rpy=-1.4614506473940839798e-15 -2.1038726316805495209e-14 -4.9960036110118277749e-16
- joint right_knee: origin xyz=-1.360023205165816762e-15 0.07864999999999899849 0.036999999999998534062 rpy=3.141592653589793116 -5.3042305426499207572e-15 1.0017539295583627067e-13 -> xyz=-2.0816681711721685133e-17 0.078649999999999151146 0.036999999999999075295 rpy=3.1415926535897922278 -4.3118451852923719846e-26 2.0787928434596164854e-13
- joint trunk_frame: origin xyz=-0.060471084556686989508 -0.0063972335546741820184 0.066744147727335195741 rpy=-6.3086333636868837384e-14 0.021825623709755163221 1.3209498708375492755e-13 -> xyz=-0.024000000000000760308 -2.4112656316077618612e-16 0.088190938812376745704 rpy=-1.4062102177136726269e-16 -9.4252837597218562265e-17 7.8061435390716270015e-33
