Commit message: new urdf and mjcf

File: mini_bdx/robots/open_duck_mini_v2/robot.urdf (robot description, URDF)
Before this commit: robot onshape, 21 links, 20 joints
Links:
- link head_assembly: mass 0.33587292587593409188 -> 0.35258298534369564292; geometry collision mesh filename=package:///board.stl; collision mesh filename=package:///drive_palonier.stl
- link head_pitch_to_yaw: mass 0.015591038955987642986 -> 0.016937787992335997383
- link hip_roll_assembly: mass 0.066480000000000025184 -> 0.06648000000000005294
- link hip_roll_assembly_2: mass 0.066480000000000025184 -> 0.06648000000000005294
- link knee_and_ankle_assembly: mass 0.12407000000000002748 -> 0.12407000000000001361
- link knee_and_ankle_assembly_2: mass 0.072590000000000029501 -> 0.072590000000000057256
- link knee_and_ankle_assembly_3: mass 0.12407000000000002748 -> 0.12407000000000001361
- link knee_and_ankle_assembly_4: mass 0.072590000000000029501 -> 0.072590000000000057256
- link left_antenna_holder: mass 0.00421628909577088061 -> 0.0042162890957708797426
- link left_roll_to_pitch_assembly: mass 0.075160000000000018461 -> 0.075160000000000060094
- link neck_pitch_assembly: mass 0.066180000000000030469 -> 0.066180000000000058225
- link neck_yaw_assembly: mass 0.090572249204174976045 -> 0.09180988857925044544
- link right_roll_to_pitch_assembly: mass 0.075160000000000032339 -> 0.075160000000000060094
- link trunk_assembly: mass 0.69443340465392744409 -> 0.69852641931996084512; geometry collision mesh filename=package:///battery_pack_lid.stl; collision mesh filename=package:///bms.stl
Joints:
- joint head_frame: origin xyz=0.042450000000000626121 -2.563053935755732482e-16 0.03595000000000117546 rpy=-1.2621774483535835759e-29 1.5707963267948756858 0 -> xyz=0.04245000000000057061 7.4178402136026999614e-16 0.035949999999999988909 rpy=2.2204460492701854731e-16 1.570796326794896336 0
- joint head_pitch: origin xyz=-5.6378512969246230568e-18 0.066000000000000003109 -6.9388939039072283776e-18 rpy=5.9571514509304171254e-17 -7.163548953726033378e-17 1.6653345369378257762e-16 -> xyz=8.6736173798840354721e-19 0.066000000000000016986 -3.4694469519536141888e-18 rpy=-1.4406834481465239151e-16 -1.1423136877781657605e-16 1.1213426021061680001e-13
- joint head_roll: origin xyz=0.040950000000000402745 1.1462727468602995629e-16 -0.019150000000000444444 rpy=-2.4980018054066286428e-15 -1.5707963267948730213 0 -> xyz=0.040950000000000097433 -1.7527483370943786056e-16 -0.019149999999999778311 rpy=-7.3227915058204641542e-14 -1.570796326794896336 0
- joint head_yaw: origin xyz=-1.5178830414797062076e-17 0.056999999999999939604 0.019049999999999959327 rpy=-1.570796326794896558 -7.286368982477690022e-17 -5.2678381782433861865e-15 -> xyz=-1.6913553890773869171e-17 0.056999999999999939604 0.019050000000000014838 rpy=-1.570796326794896558 7.3522809646371816617e-14 6.1232339957365034931e-17
- joint left_ankle: origin xyz=3.8857805861880478915e-16 -0.078649999999999067879 9.9999999999947353224e-05 rpy=-3.0577093135086125731e-16 -2.1510571099027823781e-16 -1.1379786005983670304e-15 -> xyz=-3.4694469519536141888e-17 -0.078650000000000178102 9.99999999999751088e-05 rpy=-2.6413756774523519415e-16 1.2220841311108591179e-26 2.7755576181993178136e-17
- joint left_antenna: origin xyz=0.00070406945503787010665 0.060662837687360374184 0.11643485329544565887 rpy=3.1415926535897309435 1.3045791727887228184 1.3234423712230789505 -> xyz=0.00070406945503534434927 0.060662837687359784378 0.11643485329544212004 rpy=-3.1415926535896234739 1.3045791727887248168 1.3234423712232488146
- joint left_foot_frame: origin xyz=0.00049999999999996574962 -0.036224999999999646372 0.019550000000000317124 rpy=-1.570796326794896558 4.8789097759078905605e-18 3.7865323450608544239e-29 -> xyz=0.00049999999999996574962 -0.036224999999999729638 0.01955000000000034488 rpy=-1.570796326794896558 4.8789097742003279458e-18 8.5828066488045564267e-28
- joint left_hip_pitch: origin xyz=0.074149999999998994493 5.7702594872394152858e-16 0.035109999999999731701 rpy=-3.141592653589793116 1.5707963267948958919 0 -> xyz=0.074149999999999799405 1.3959102970750869588e-18 0.035109999999999912113 rpy=3.141592653589793116 1.5707963267948952257 0
- joint left_hip_roll: origin xyz=0.019050000000002908357 -1.2559397966072083364e-15 -0.046015000000000465252 rpy=-1.57079632679495651 1.0208316397064496209e-13 1.5707963267945266317 -> xyz=0.019050000000003241424 2.0469737016526323714e-15 -0.046015000000000895464 rpy=-1.5707963267949442976 1.0251581517556108667e-13 1.5707963267946023489
- joint left_hip_yaw: origin xyz=-0.018999999999999715034 0.035000000000001356415 0.045940938812377457579 rpy=-5.4063708435955792693e-16 -2.1649348979904514729e-14 -1.6653345373435771223e-16 -> xyz=-0.019000000000000290962 0.035000000000001273148 0.045940938812378845357 rpy=-2.0757017677015319346e-16 -2.1982415887547258194e-14 -7.6136910267405882653e-27
- joint left_knee: origin xyz=6.2450045135165055399e-17 -0.078649999999999636868 9.9999999999988986588e-05 rpy=-1.433738720798104591e-17 9.7838404045009444717e-16 4.9960036108120734026e-16 -> xyz=1.3877787807814456755e-17 -0.078650000000000011569 9.9999999999961231012e-05 rpy=-2.6413756781799972404e-16 -2.7339812777890022088e-26 0
- joint neck_pitch: origin xyz=0.00099999999999897046243 0.019150000000000326483 0.090000938812376238274 rpy=1.57079632679489678 -2.2148949341271863515e-14 2.5552148182455563673e-16 -> xyz=0.00099999999999896352354 0.019150000000000326483 0.090000938812376238274 rpy=1.570796326794896558 8.9928064994637667153e-14 6.1232449686014378908e-17
- joint right_ankle: origin xyz=-2.5673907444456744997e-16 -0.078649999999999331557 9.9999999999947353224e-05 rpy=3.1786111035240684541e-16 -6.6613381497353178635e-16 1.026830726893522614e-13 -> xyz=-6.9388939039072283776e-18 -0.078650000000000039324 9.9999999999961231012e-05 rpy=-2.6413756984180028828e-16 -6.9382288127881716121e-25 -5.1722034616178551878e-17
- joint right_antenna: origin xyz=0.00070406945503653783902 -0.060662837687360852967 0.11643485329544586704 rpy=-3.1415926535897518157 1.3045791727887290357 -1.3234423712230898307 -> xyz=0.00070406945503534434927 -0.06066283768735826476 0.11643485329544212004 rpy=3.1415926535896230298 1.3045791727887245948 -1.3234423712232490367
- joint right_foot_frame: origin xyz=0.00050000000000024330538 -0.036224999999999923928 0.019550000000000650191 rpy=-1.570796326794896558 -3.0222156344620005664e-28 -2.5243548967072377773e-28 -> xyz=0.0005000000000002155498 -0.036224999999999840661 0.019550000000000664069 rpy=-1.570796326794896558 9.1691846176123393012e-16 1.3322725304659061714e-15
- joint right_hip_pitch: origin xyz=-0.074149999999999938183 1.3700249702069955404e-16 0.035109999999999981501 rpy=-5.8199867801976243694e-16 1.5707963267947913089 0 -> xyz=-0.074149999999999799405 3.1868767607495795957e-16 0.035110000000000016196 rpy=-2.3836094894413110414e-24 1.570796326794896336 0
- joint right_hip_roll: origin xyz=0.019050000000007772522 3.498590306350024548e-14 -0.046015000000001887726 rpy=-1.5707963267947930852 -7.5380278374294396407e-14 1.5707963267945495023 -> xyz=0.019050000000008261714 3.78516662458139308e-14 -0.046015000000003032643 rpy=-1.5707963267947879782 -8.4491074221037422062e-14 1.5707963267945974639
- joint right_hip_yaw: origin xyz=-0.018999999999999697686 -0.035000000000001127431 0.045940938812377443701 rpy=-1.4614506473940839798e-15 -2.1038726316805495209e-14 -4.9960036110118277749e-16 -> xyz=-0.018999999999998431338 -0.03500000000000151601 0.045940938812377415945 rpy=-4.6224992538811313716e-16 -2.2037927038832600325e-14 -1.6653345370219725828e-16
- joint right_knee: origin xyz=-2.0816681711721685133e-17 0.078649999999999151146 0.036999999999999075295 rpy=3.1415926535897922278 -4.3118451852923719846e-26 2.0787928434596164854e-13 -> xyz=-6.9388939039072283776e-18 0.078649999999999414824 0.036999999999999658162 rpy=3.141592653589793116 -2.0819102970830263503e-24 5.0289882707839502595e-30
